File: KiCad_Project/tempsensor.kicad_pcb (KiCad board)
At the start: 2 copper layers, 32.2 x 43.2 mm, 37 parts, among them J1 Conn_01x01_Male, J2 SWD, J3 WD_Disable, J4 Conn_01x01_Male, J5 Conn_01x01_Male, J6 Conn_01x01_Male, Q1 BSS84, U1 STM32F303K8Tx, U2 UJA1075A, U3 MLX90614ESF-BAA-000-TU, Y1 8Mhz

Commit message: Updated board traces
Parts:
- 12V: renamed from J1; footprint MountingHole:MountingHole_2.2mm_M2_Pad_Via -> Connector_PinHeader_2.54mm:PinHeader_1x01_P2.54mm_Vertical
- CANH: renamed from J5; footprint MountingHole:MountingHole_2.2mm_M2_Pad_Via -> Connector_PinHeader_2.54mm:PinHeader_1x01_P2.54mm_Vertical
- CANL: renamed from J6; footprint MountingHole:MountingHole_2.2mm_M2_Pad_Via -> Connector_PinHeader_2.54mm:PinHeader_1x01_P2.54mm_Vertical
- GND: renamed from J4; footprint MountingHole:MountingHole_2.2mm_M2_Pad_Via -> Connector_PinHeader_2.54mm:PinHeader_1x01_P2.54mm_Vertical
- moved GND 3.42 mm to (90.8, 32.4)
- moved CANH 2.84 mm to (106.0, 32.4)
- moved R9 2.01 mm to (106.0, 50.8)
- moved 12V 1.80 mm to (95.9, 32.4)
- moved CANL 1.42 mm to (101.0, 32.4)
- moved C2 1.27 mm to (88.3, 54.6)
Routing:
- net +3V3: track 0.00 -> 104.6 mm, vias 0 -> 5
- net RESET: track 0.00 -> 33.8 mm, vias 0 -> 4
- net +12V: track 0.00 -> 17.6 mm
- net CAN_RX: track 0.00 -> 17.3 mm, vias 0 -> 2
- net I2C_SDA: track 0.00 -> 16.4 mm
- net CAN_TX: track 0.00 -> 15.9 mm, vias 0 -> 2
- net GND: track 0.00 -> 15.8 mm, vias 0 -> 4
- net I2C_SCL: track 0.00 -> 14.7 mm
- net SWDIO: track 0.00 -> 12.3 mm, vias 0 -> 1
- net TDI: track 0.00 -> 12.0 mm, vias 0 -> 1
- net SWDCLK: track 0.00 -> 11.2 mm, vias 0 -> 1
- net PA8: track 0.00 -> 11.2 mm
- net SWO: track 0.00 -> 10.9 mm
- net CANH: track 0.00 -> 10.9 mm
- net CANL: track 0.00 -> 9.70 mm
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Other:
- board size 32.2 x 43.2 mm -> 32.2 x 41.9 mm

Commit message: Final Version
Parts:
- moved D5 5.43 mm to (87.6, 64.1)
- moved R12 5.43 mm to (89.5, 64.1)
- moved D2 5.08 mm to (89.5, 58.4)
- moved R10 5.08 mm to (87.6, 58.4)
Routing:
- net PA8: track 11.2 -> 6.09 mm
- net CAN_TX: track 15.9 -> 19.9 mm
- net CAN_RX: track 17.3 -> 20.4 mm
- net SWO: track 10.9 -> 7.84 mm, vias 0 -> 1
- net TDI: track 12.0 -> 9.31 mm
- net GND: track 15.8 -> 14.4 mm, vias 4 -> 8
- net SWDCLK: track 11.2 -> 10.1 mm
- net CANL: track 9.70 -> 9.06 mm
- net I2C_SCL: track 14.7 -> 14.0 mm
- net +3V3: track 104.6 -> 104.4 mm, vias 5 -> 4
Other:
- board text added: "Tire Temp Sensor V1 MB Joel Sol 10/20"
