File: KiCad_Project/tempsensor.sch (KiCad schematic (older format))
At the start: 37 parts, among them J1 Conn_01x01_Male, J2 SWD, J3 WD_Disable, J4 Conn_01x01_Male, J5 Conn_01x01_Male, J6 Conn_01x01_Male, Q1 BSS84, U1 STM32F303K8Tx, U2 UJA1075A, U3 MLX90614ESF-BAA-000-TU, Y1 8Mhz

Commit message: Updated board traces
Other:
- note added: "Infrared Tire Temperature Sensor"
- note added: "Joel Sol"
- note added: "Oct 21 2020"
Changed lines of the file:
@@
 Text Notes 2450 5700 0    50   ~ 0
 Ext. Oscillator
+Text Notes 12200 10900 0    50   ~ 0
+Infrared Tire Temperature Sensor
+Text Notes 13000 11050 0    50   ~ 0
+Oct 21 2020
+Text Notes 11900 10500 0    50   ~ 0
+Joel Sol
 $EndSCHEMATC

Commit message: update
Other:
- note removed: "Infrared Tire Temperature Sensor"
- note removed: "Joel Sol"
- note removed: "Oct 21 2020"
- moved on the sheet: C1, C10, C2, C3, C4, C6, C7, C8, C9, D1, D2, D4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
